File: Nivara_PCB/ANALOG_IN.kicad_sch (KiCad schematic)
At the start: 5 parts

Commit message: Cambios realizados en los archivos de Nivara_PCB.
Parts:
- C10: symbol PCM_Capacitor_US_AKL:C_0603 -> EasyEDA:C_0603
- D17, D18: symbol PCM_Diode_TVS_AKL:SMAJ5.0A -> EasyEDA:SMAJ5.0A
- R21: symbol PCM_Resistor_US_AKL:R_0603 -> EasyEDA:R_0603
- R22: symbol PCM_Resistor_US_AKL:R_0805 -> EasyEDA:R_0805
Changed lines of the file:
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@@
 	)
 	(symbol
-		(lib_id "PCM_Capacitor_US_AKL:C_0603")
+		(lib_id "EasyEDA:C_0603")
 		(at 60.96 67.31 0)
 		(unit 1)
@@
 	)
 	(symbol
-		(lib_id "PCM_Resistor_US_AKL:R_0805")
+		(lib_id "EasyEDA:R_0805")
 		(at 72.39 66.04 0)
 		(unit 1)
@@
 	)
 	(symbol
-		(lib_id "PCM_Diode_TVS_AKL:SMAJ5.0A")
+		(lib_id "EasyEDA:SMAJ5.0A")
 		(at 55.88 67.31 270)
 		(mirror x)
@@
 	)
 	(symbol
-		(lib_id "PCM_Diode_TVS_AKL:SMAJ5.0A")
+		(lib_id "EasyEDA:SMAJ5.0A")
 		(at 55.88 53.34 270)
 		(mirror x)
@@
 	)
 	(symbol
-		(lib_id "PCM_Resistor_US_AKL:R_0603")
+		(lib_id "EasyEDA:R_0603")
 		(at 66.04 59.69 90)
 		(unit 1)
@@
 	)
 	(symbol
-		(lib_id "power:+3.3V")
+		(lib_id "EasyEDA:+3.3V")
 		(at 55.88 46.99 0)
 		(unit 1)
@@
 	)
 	(symbol
-		(lib_id "power:GND")
+		(lib_id "EasyEDA:GND")
 		(at 72.39 76.2 0)
 		(unit 1)
