File: Nivara_PCB/D_IN.kicad_sch (KiCad schematic)
At the start: 4 parts, among them U12 LTV-357T

Commit message: Cambios realizados en los archivos de Nivara_PCB.
Parts:
- D20: symbol Device:LED -> EasyEDA:LED
- R27, R28: symbol PCM_Resistor_US_AKL:R_0603 -> EasyEDA:R_0603
- U12: symbol Isolator:LTV-357T -> EasyEDA:LTV-357T
Changed lines of the file:
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@@
 	)
 	(symbol
-		(lib_id "PCM_Resistor_US_AKL:R_0603")
+		(lib_id "EasyEDA:R_0603")
 		(at 76.2 53.34 0)
 		(unit 1)
@@
 	)
 	(symbol
-		(lib_id "power:GND")
+		(lib_id "EasyEDA:GND")
 		(at 54.61 81.28 0)
 		(unit 1)
@@
 	)
 	(symbol
-		(lib_id "Device:LED")
+		(lib_id "EasyEDA:LED")
 		(at 76.2 62.23 90)
 		(unit 1)
@@
 	)
 	(symbol
-		(lib_id "power:GND")
+		(lib_id "EasyEDA:GND")
 		(at 76.2 81.28 0)
 		(unit 1)
@@
 	)
 	(symbol
-		(lib_id "Isolator:LTV-357T")
+		(lib_id "EasyEDA:LTV-357T")
 		(at 66.04 74.93 0)
 		(unit 1)
@@
 	)
 	(symbol
-		(lib_id "PCM_Resistor_US_AKL:R_0603")
+		(lib_id "EasyEDA:R_0603")
 		(at 54.61 52.07 0)
 		(unit 1)
@@
 	)
 	(symbol
-		(lib_id "power:+3.3V")
+		(lib_id "EasyEDA:+3.3V")
 		(at 76.2 46.99 0)
 		(unit 1)
