File: Nivara_PCB/NIVARA_BOARD.kicad_sch (KiCad schematic)
At the start: 5 parts, among them U3 ESP32-S3-WROOM-1

Commit message: Cambios realizados en los archivos de Nivara_PCB.
Parts:
- C2, C3: symbol PCM_Capacitor_US_AKL:C_0603 -> EasyEDA:C_0603
- R1, R2: symbol PCM_Resistor_US_AKL:R_0603 -> EasyEDA:R_0603
- U3: symbol PCM_Espressif:ESP32-S3-WROOM-1 -> EasyEDA:ESP32-S3-WROOM-1
Changed lines of the file:
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@@
 	)
 	(symbol
-		(lib_id "power:+3.3V")
+		(lib_id "EasyEDA:+3.3V")
 		(at 137.16 55.88 0)
 		(unit 1)
@@
 	)
 	(symbol
-		(lib_id "PCM_Espressif:ESP32-S3-WROOM-1")
+		(lib_id "EasyEDA:ESP32-S3-WROOM-1")
 		(at 137.16 99.06 0)
 		(unit 1)
@@
 	)
 	(symbol
-		(lib_id "PCM_Resistor_US_AKL:R_0603")
+		(lib_id "EasyEDA:R_0603")
 		(at 189.23 127 90)
 		(mirror x)
@@
 	)
 	(symbol
-		(lib_id "PCM_Capacitor_US_AKL:C_0603")
+		(lib_id "EasyEDA:C_0603")
 		(at 48.26 36.83 0)
 		(mirror y)
@@
 	)
 	(symbol
-		(lib_id "power:GND")
+		(lib_id "EasyEDA:GND")
 		(at 137.16 142.24 0)
 		(unit 1)
@@
 	)
 	(symbol
-		(lib_id "PCM_Resistor_US_AKL:R_0603")
+		(lib_id "EasyEDA:R_0603")
 		(at 185.42 140.97 0)
 		(mirror y)
@@
 	)
 	(symbol
-		(lib_id "PCM_Capacitor_US_AKL:C_0603")
+		(lib_id "EasyEDA:C_0603")
 		(at 78.74 36.83 0)
 		(mirror y)
@@
 	)
 	(symbol
-		(lib_id "power:+3.3V")
+		(lib_id "EasyEDA:+3.3V")
 		(at 78.74 29.21 0)
 		(unit 1)
@@
 	)
 	(symbol
-		(lib_id "power:GND")
+		(lib_id "EasyEDA:GND")
 		(at 78.74 43.18 0)
 		(unit 1)
@@
 	)
 	(symbol
-		(lib_id "power:+3.3V")
+		(lib_id "EasyEDA:+3.3V")
 		(at 48.26 29.21 0)
 		(unit 1)
@@
 	)
 	(symbol
-		(lib_id "power:GND")
+		(lib_id "EasyEDA:GND")
 		(at 48.26 43.18 0)
 		(unit 1)
