File: Nivara_PCB/Nivara_PCB.kicad_sch (KiCad schematic)
At the start: 21 parts, among them CN1 ANALOG_IN, CN2 RELAY, J1 AUXILIAR, P1 NPN_IN, P2 PNP_IN, P3 D_IN, P4 RUN/STOP, P5 NPN_OUT, P6 PNP_OUT, P7 RS485, P8 ANALOG_OUT., U1 2.54-2*2, U2 FUENTE IN

Commit message: Changes en diseño.
Connections:
- net GND1 is gone; now on net GND: D3.2 (A), H1.1, H2.1, U2.2
Other:
- moved on the sheet: D3
Changed lines of the file:
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@@
 	(wire
 		(pts
-			(xy 213.36 66.04) (xy 213.36 74.93)
+			(xy 213.36 66.04) (xy 213.36 71.12)
 		)
 		(stroke
@@
 	(wire
 		(pts
-			(xy 213.36 85.09) (xy 213.36 82.55)
+			(xy 213.36 81.28) (xy 213.36 78.74)
 		)
 		(stroke
@@
 	(symbol
 		(lib_id "EasyEDA:GND")
-		(at 213.36 85.09 0)
-		(unit 1)
-		(exclude_from_sim no)
-		(in_bom yes)
-		(on_board yes)
-		(dnp no)
-		(fields_autoplaced yes)
+		(at 213.36 81.28 0)
+		(unit 1)
+		(exclude_from_sim no)
+		(in_bom yes)
+		(on_board yes)
+		(dnp no)
 		(property "Reference" "#PWR012"
-			(at 213.36 91.44 0)
-			(effects
-				(font
-					(size 1.27 1.27)
-				)
-				(hide yes)
-			)
-		)
-		(property "Value" "GND1"
-			(at 213.36 90.17 0)
-			(effects
-				(font
-					(size 1.27 1.27)
-				)
+			(at 213.36 87.63 0)
+			(effects
+				(font
+					(size 1.27 1.27)
+				)
+				(hide yes)
+			)
+		)
+		(property "Value" "GND"
+			(at 211.582 85.852 0)
+			(effects
+				(font
+					(size 1.27 1.27)
+				)
+				(justify left)
 			)
 		)
 		(property "Footprint" ""
-			(at 213.36 85.09 0)
+			(at 213.36 81.28 0)
 			(effects
 				(font
@@
 		)
 		(property "Datasheet" ""
-			(at 213.36 85.09 0)
+			(at 213.36 81.28 0)
 			(effects
 				(font
@@
 		)
 		(property "Description" "Power symbol creates a global label with name \"GND\" , ground"
-			(at 213.36 85.09 0)
+			(at 213.36 81.28 0)
 			(effects
 				(font
@@
 		(on_board yes)
 		(dnp no)
-		(fields_autoplaced yes)
 		(property "Reference" "#PWR09"
 			(at 198.12 77.47 0)
@@
 			)
 		)
-		(property "Value" "GND1"
-			(at 198.12 76.2 0)
-			(effects
-				(font
-					(size 1.27 1.27)
-				)
+		(property "Value" "GND"
+			(at 196.342 75.692 0)
+			(effects
+				(font
+					(size 1.27 1.27)
+				)
+				(justify left)
 			)
 		)
@@
 			)
 		)
-		(property "Value" "GND1"
-			(at 209.55 124.46 0)
-			(effects
-				(font
-					(size 1.27 1.27)
-				)
+		(property "Value" "GND"
+			(at 212.09 120.6499 0)
+			(effects
+				(font
+					(size 1.27 1.27)
+				)
+				(justify left)
 			)
 		)
@@
 	(symbol
 		(lib_id "EasyEDA:SMAJ33A")
-		(at 213.36 78.74 90)
+		(at 213.36 74.93 90)
 		(unit 1)
 		(exclude_from_sim no)
@@
 		(fields_autoplaced yes)
 		(property "Reference" "D3"
-			(at 215.9 77.4699 90)
+			(at 215.9 73.6599 90)
 			(effects
 				(font
@@
 		)
 		(property "Value" "SMAJ33A"
-			(at 215.9 80.0099 90)
+			(at 215.9 76.1999 90)
 			(effects
 				(font
@@
 		)
 		(property "Footprint" "PCM_Diode_SMD_AKL:D_SMA"
-			(at 213.36 78.74 0)
+			(at 213.36 74.93 0)
 			(effects
 				(font
@@
 		)
 		(property "Datasheet" "https://www.tme.eu/Document/dbc72d81c249fe51b6ab42300e8e06d0/SMAJ_ser.pdf"
-			(at 213.36 78.74 0)
+			(at 213.36 74.93 0)
 			(effects
 				(font
@@
 		)
 		(property "Description" "SMA Unidirectional TVS diode, 33V, 400W, Alternate KiCAD Library"
-			(at 213.36 78.74 0)
+			(at 213.36 74.93 0)
 			(effects
 				(font
@@
 			)
 		)
-		(property "Value" "GND1"
-			(at 184.15 124.46 0)
-			(effects
-				(font
-					(size 1.27 1.27)
-				)
-			)
-		)
+		(property "Value" "GND"
+			(at 186.69 120.6499 0)
+			(effects
+				(font
+					(size 1.27 1.27)
+				)
+				(justify left)
+			)
+		)

Commit message: cAMBIOS EN EL PCB Y ESQUEMA.
Connections:
- net VIN: now reaches F1.1, U2.1
Changed lines of the file:
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@@
+		)
+	)
+	(label "VIN"
+		(at 195.58 66.04 0)
+		(effects
+			(font
+				(size 1.27 1.27)
+			)
+			(justify left bottom)
 		)
 	)
