File: Nivara_PCB/PowerSupply.kicad_sch (KiCad schematic)
At the start: 19 parts, among them U4 AP63200WU

Commit message: Cambios realizados en los archivos de Nivara_PCB.
Parts:
- C4: symbol PCM_Capacitor_AKL:C_1206 -> EasyEDA:C_1206
- C5, C6: symbol PCM_Capacitor_AKL:C_0805 -> EasyEDA:C_0805
- C7, C8: symbol PCM_Capacitor_AKL:C_0603 -> EasyEDA:C_0603
- D4, D5: symbol Device:LED -> EasyEDA:LED
- JP1: symbol Jumper:SolderJumper_2_Open -> EasyEDA:SolderJumper_2_Open
- R3, R4, R5, R6: symbol PCM_Resistor_US_AKL:R_0603 -> EasyEDA:R_0603
- TP1, TP2, TP3, TP4, TP5: symbol Connector:TestPoint_Probe -> EasyEDA:TestPoint_Probe
- U4: symbol Regulator_Switching:AP63200WU -> EasyEDA:AP63200WU
Changed lines of the file:
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@@
 	)
 	(symbol
-		(lib_id "PCM_Resistor_US_AKL:R_0603")
+		(lib_id "EasyEDA:R_0603")
 		(at 161.29 63.5 180)
 		(unit 1)
@@
 	)
 	(symbol
-		(lib_id "Connector:TestPoint_Probe")
+		(lib_id "EasyEDA:TestPoint_Probe")
 		(at 96.52 69.85 0)
 		(unit 1)
@@
 	)
 	(symbol
-		(lib_id "PCM_Capacitor_AKL:C_1206")
+		(lib_id "EasyEDA:C_1206")
 		(at 53.34 58.42 0)
 		(unit 1)
@@
 	)
 	(symbol
-		(lib_id "PCM_Resistor_US_AKL:R_0603")
+		(lib_id "EasyEDA:R_0603")
 		(at 43.18 68.58 180)
 		(unit 1)
@@
 	)
 	(symbol
-		(lib_id "Connector:TestPoint_Probe")
+		(lib_id "EasyEDA:TestPoint_Probe")
 		(at 161.29 40.64 0)
 		(unit 1)
@@
 	)
 	(symbol
-		(lib_id "Regulator_Switching:AP63200WU")
+		(lib_id "EasyEDA:AP63200WU")
 		(at 71.12 49.53 0)
 		(unit 1)
@@
 	)
 	(symbol
-		(lib_id "Device:LED")
+		(lib_id "EasyEDA:LED")
 		(at 43.18 58.42 90)
 		(unit 1)
@@
 	)
 	(symbol
-		(lib_id "PCM_Capacitor_AKL:C_0603")
+		(lib_id "EasyEDA:C_0603")
 		(at 142.24 58.42 0)
 		(unit 1)
@@
 	)
 	(symbol
-		(lib_id "Connector:TestPoint_Probe")
+		(lib_id "EasyEDA:TestPoint_Probe")
 		(at 142.24 40.64 0)
 		(unit 1)
@@
 	)
 	(symbol
-		(lib_id "PCM_Resistor_US_AKL:R_0603")
+		(lib_id "EasyEDA:R_0603")
 		(at 118.11 53.34 0)
 		(unit 1)
@@
 	)
 	(symbol
-		(lib_id "PCM_Capacitor_AKL:C_0603")
+		(lib_id "EasyEDA:C_0603")
 		(at 129.54 58.42 0)
 		(unit 1)
@@
 	)
 	(symbol
-		(lib_id "power:GND")
+		(lib_id "EasyEDA:GND")
 		(at 71.12 76.2 0)
 		(unit 1)
@@
 	)
 	(symbol
-		(lib_id "Device:LED")
+		(lib_id "EasyEDA:LED")
 		(at 161.29 53.34 90)
 		(unit 1)
@@
 	)
 	(symbol
-		(lib_id "PCM_Resistor_US_AKL:R_0603")
+		(lib_id "EasyEDA:R_0603")
 		(at 118.11 66.04 0)
 		(unit 1)
@@
 	)
 	(symbol
-		(lib_id "PCM_Capacitor_AKL:C_0805")
+		(lib_id "EasyEDA:C_0805")
 		(at 87.63 49.53 90)
 		(unit 1)
@@
 	)
 	(symbol
-		(lib_id "power:+3.3V")
+		(lib_id "EasyEDA:+3.3V")
 		(at 177.8 41.91 0)
 		(unit 1)
@@
 	)
 	(symbol
-		(lib_id "power:VCC")
+		(lib_id "EasyEDA:VCC")
 		(at 43.18 43.18 0)
 		(unit 1)
@@
 	)
 	(symbol
-		(lib_id "Jumper:SolderJumper_2_Open")
+		(lib_id "EasyEDA:SolderJumper_2_Open")
 		(at 152.4 46.99 0)
 		(unit 1)
@@
 	)
 	(symbol
-		(lib_id "Connector:TestPoint_Probe")
+		(lib_id "EasyEDA:TestPoint_Probe")
 		(at 96.52 57.15 0)
 		(unit 1)
@@
 	)
 	(symbol
-		(lib_id "Connector:TestPoint_Probe")
+		(lib_id "EasyEDA:TestPoint_Probe")
 		(at 53.34 41.91 0)
 		(unit 1)
@@
 	)
 	(symbol
-		(lib_id "PCM_Capacitor_AKL:C_0805")
+		(lib_id "EasyEDA:C_0805")
 		(at 107.95 53.34 180)
 		(unit 1)

Commit message: cAMBIOS EN EL PCB Y ESQUEMA.
Connections:
- net FB: now reaches C6.1, R4.2, R5.1, TP2.1, U4.1 (FB)
- net SW: now reaches C5.2, L1.1, U4.5 (SW)
- net BST: now reaches C5.1, U4.6 (BST)
- net VOUT: now reaches C6.2, C7.1, C8.1, JP1.1 (A), L1.2, R4.1, TP4.1
Changed lines of the file:
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@@
+		)
+	)
+	(label "VOUT"
+		(at 120.65 46.99 0)
+		(effects
+			(font
+				(size 1.27 1.27)
+			)
+			(justify left bottom)
+		)
+	)
+	(label "BST"
+		(at 82.55 49.53 0)
+		(effects
+			(font
+				(size 1.27 1.27)
+			)
+			(justify left bottom)
+		)
+	)
+	(label "FB"
+		(at 100.33 59.69 0)
+		(effects
+			(font
+				(size 1.27 1.27)
+			)
+			(justify left bottom)
+		)
+	)
+	(label "SW"
+		(at 90.17 46.99 0)
+		(effects
+			(font
+				(size 1.27 1.27)
+			)
+			(justify left bottom)
 		)
 	)
