File: Nivara_PCB/Nivara_PCB/Nivara_PCB.kicad_pcb (KiCad board)
At the start: 4 copper layers, 98.8 x 81.2 mm, 162 parts, among them CN1 ANALOG_IN, CN2 RELAY, J1 AUXILIAR, K1 SRA-24VDC-CL, K2 SRA-24VDC-CL, P1 NPN_IN, P2 PNP_IN, P3 D_IN, P4 RUN/STOP, P5 NPN_OUT, P6 PNP_OUT, P7 RS485, P8 ANALOG_OUT., Q1 IRLML0040, Q2 AO3407A, Q3 IRLML0040, Q4 AO3407A, Q5 IRLML6402TRPBF-JSM, SW1 SKRPACE010, SW2 SKRPACE010, U1 2.54-2*2, U10 GP8201S-TC50-EW, U11 LK1802, U12 LTV-357T, U13 LTV-357T, U14 LTV-357T, U15 LTV-357T, U16 LTV-357T, U17 LTV-357T, U18 LTV-357T, U19 GP8303-TC50-EW, U2 FUENTE IN, U3 ESP32-S3-WROOM-1, U4 AP63200WU, U5 RSM3485ECHT_C2992406, U6 LTV-357T, U7 LTV-357T, U8 LTV-357T, U9 LTV-357T

Commit message: Saved changes to Nivara PCB files
Parts:
- removed D12, D21: PMEG4010CEH, PCM_Diode_SMD_AKL:D_SOD-123F
- removed D34: SMAJ5.0A, PCM_Diode_SMD_AKL:D_SMA
- added C20: 1uF, PCM_Capacitor_SMD_AKL:C_0603_1608Metric, F.Cu at (187.9, 97.2)
- added D29: SMF5.0A, SMF5.0A:SODFL3718X102N, F.Cu at (233.4, 54.3)
- added D30: SMF5.0A, SMF5.0A:SODFL3718X102N, F.Cu at (248.1, 55.7)
- added F2: BSMD1812-150-33V, EasyEDA:F1812, F.Cu at (254.8, 51.2)
- added R58: 22k, PCM_Resistor_SMD_AKL:R_0603_1608Metric, F.Cu at (183.9, 90.4)
- added R59: 22k, PCM_Resistor_SMD_AKL:R_0603_1608Metric, F.Cu at (182.1, 90.4)
- added R60: 22k, PCM_Resistor_SMD_AKL:R_0603_1608Metric, F.Cu at (187.9, 99.2)
- added U20: FUENTE EX, EasyEDA:CONN-TH_XY126V-5.0-2P, F.Cu at (257.2, 43.8)
- D17, D18, D31, D32: value SMAJ5.0A -> SMF5.0A; footprint PCM_Diode_SMD_AKL:D_SMA -> SMF5.0A:SODFL3718X102N
- D33: value SMAJ5.0A -> SMAJ33A
- R15, R31: value 20k -> 30k
- moved C2 151.9 mm to (243.6, 80.9)
- moved C3 151.9 mm to (243.6, 83.6)
- moved R1 151.9 mm to (243.5, 75.4)
- moved R2 151.9 mm to (243.5, 78.2)
- moved R38 144.9 mm to (244.8, 100.0), turned to 90 degrees
- moved R40 143.7 mm to (243.8, 108.8), turned to 180 degrees
- moved R39 142.9 mm to (242.8, 102.0), turned to 90 degrees
- moved R37 142.7 mm to (242.0, 90.2)
- moved Q4 140.3 mm to (244.8, 105.8), turned to -90 degrees
- moved U16 135.1 mm to (241.8, 95.6), turned to -90 degrees
- moved D27 133.6 mm to (243.4, 111.6), turned to 180 degrees
- moved D28 131.2 mm to (240.8, 107.8), turned to 90 degrees
- moved R16 127.1 mm to (227.1, 105.5), turned to -90 degrees
- moved R15 127.1 mm to (227.2, 100.4), turned to 90 degrees
- moved D2 126.7 mm to (262.0, 74.9), turned to 90 degrees
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Connections:
- D13 pad 1: VCC -> VDD
- D13 pad 2: /NIVARA_BOARD/NPN_OUT_1/NPN_OUT -> /NIVARA_BOARD/NPN_OUT_1
- D14 pad 1: /NIVARA_BOARD/NPN_OUT_1/NPN_OUT -> /NIVARA_BOARD/NPN_OUT_1
- D15 pad 2: GND -> Earth
- D16 pad 1: GND -> Earth
- D22 pad 1: VCC -> VDD
- D22 pad 2: /NIVARA_BOARD/NPN_OUT_2/NPN_OUT -> /NIVARA_BOARD/NPN_OUT_2
- D23 pad 1: /NIVARA_BOARD/NPN_OUT_2/NPN_OUT -> /NIVARA_BOARD/NPN_OUT_2
- D27 pad 2: GND -> Earth
- D28 pad 1: GND -> Earth
- D33 pad 1: +3.3V -> VDD
- D33 pad 2: /NIVARA_BOARD/A_0-10_IN/A_V_OUT -> Earth
- P4 pad 2: GND -> Earth
- Q1 pad 2: GND -> Earth
- Q1 pad 3: /NIVARA_BOARD/NPN_OUT_1/NPN_OUT -> /NIVARA_BOARD/NPN_OUT_1
- Q2 pad 2: VCC -> VDD
- Q3 pad 2: GND -> Earth
- Q3 pad 3: /NIVARA_BOARD/NPN_OUT_2/NPN_OUT -> /NIVARA_BOARD/NPN_OUT_2
- Q4 pad 2: VCC -> VDD
- R11 pad 1: VCC -> VDD
- R13 pad 1: /NIVARA_BOARD/NPN_OUT_1 -> /NIVARA_BOARD/NPN_OUT_1/NPN_IN
- R14 pad 2: GND -> Earth
- R15 pad 1: VCC -> VDD
- R16 pad 1: VCC -> VDD
- R19 pad 1: VCC -> VDD
- R27 pad 1: /NIVARA_BOARD/D_IN_1 -> VDD
- R29 pad 1: /NIVARA_BOARD/NPN_OUT_2 -> /NIVARA_BOARD/NPN_OUT_2/NPN_IN
- R30 pad 2: GND -> Earth
- R31 pad 1: VCC -> VDD
- R32 pad 1: VCC -> VDD
- R35 pad 1: VCC -> VDD
- R39 pad 1: VCC -> VDD
- R41 pad 1: /NIVARA_BOARD/D_IN_2 -> VDD
- R43 pad 1: /NIVARA_BOARD/RUN/STOP -> VDD
- U12 pad 2: GND -> /NIVARA_BOARD/D_IN_1
- U14 pad 2: GND -> Earth
- U16 pad 3: GND -> Earth
- U17 pad 2: GND -> /NIVARA_BOARD/D_IN_2
- U18 pad 2: GND -> /NIVARA_BOARD/RUN/STOP
- U19 pad 10: unconnected-(U19-V5V-Pad10) -> Net-(U19-V5V)
- U19 pad 11: unconnected-(U19-EP-Pad11) -> GND
- U19 pad 3: unconnected-(U19-A0-Pad3) -> Net-(U19-A0)
- U19 pad 4: unconnected-(U19-A1-Pad4) -> Net-(U19-A1)
- U19 pad 9: unconnected-(U19-A2-Pad9) -> Net-(U19-A2)
- U3 pad 34: /NIVARA_BOARD/NPN_OUT_1/NPN_OUT -> /NIVARA_BOARD/NPN_OUT_1/NPN_IN
- U3 pad 35: /NIVARA_BOARD/NPN_OUT_2/NPN_OUT -> /NIVARA_BOARD/NPN_OUT_2/NPN_IN
- U6 pad 2: GND -> Earth
- U9 pad 3: GND -> Earth
Routing:
- net VCC: track 205.1 -> 116.2 mm, vias 24 -> 23
- net Earth: track 0.00 -> 34.5 mm, vias 0 -> 131
- net /NIVARA_BOARD/PNP_OUT_2: track 0.00 -> 13.6 mm
- net /NIVARA_BOARD/NPN_OUT_2: track 0.00 -> 13.0 mm
- net /NIVARA_BOARD/NPN_OUT_1: track 0.00 -> 12.9 mm
- net /NIVARA_BOARD/PNP_OUT_1: track 0.00 -> 12.5 mm
- net Net-(D36-K): track 0.00 -> 11.2 mm
- net /NIVARA_BOARD/I_OUT: track 0.00 -> 8.82 mm
- net +3.3V: track 0.00 -> 8.40 mm, vias 108 -> 114
- net VDD: track 0.00 -> 8.36 mm, vias 0 -> 91
- net Net-(Q4-G): track 0.00 -> 6.14 mm
- net Net-(Q3-G): track 0.00 -> 6.07 mm
- net Net-(D35-A): track 0.00 -> 5.99 mm
- net Net-(Q1-G): track 0.00 -> 5.63 mm
- net Net-(D16-A): track 0.00 -> 5.14 mm
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- added copper zone on F.Cu, net Earth
- added copper zone on In1.Cu, net Earth
- added copper zone on F.Cu, net Net-(F2-Pad1)
- added copper zone on B.Cu, net VDD
- added copper zone on F.Cu, net VDD
- removed copper zone on B.Cu, net GND

Commit message: Cambios en la salida de corriente de la PCB Nivara
Routing:
- net VCC: track 116.2 -> 119.0 mm
- net GND: vias 217 -> 239
- net +3.3V: vias 114 -> 112

Commit message: PCB casi terminado.
Parts:
- removed D26, D39: IR26-21C_L110_TR8, LED_SMD:LED_1206_3216Metric
- added D12: IR26-21C_L110_TR8, LED_SMD:LED_1206_3216Metric, F.Cu at (225.7, 62.0)
- added D21: IR26-21C_L110_TR8, LED_SMD:LED_1206_3216Metric, F.Cu at (208.8, 62.2)
- moved C15 125.1 mm to (258.7, 110.2), turned to -90 degrees
- moved R49 122.9 mm to (260.6, 111.1), turned to -90 degrees
- moved SW1 120.5 mm to (254.7, 110.6)
- moved C16 107.7 mm to (249.5, 73.0)
- moved U5 107.3 mm to (213.8, 77.4), turned to -90 degrees
- moved R50 104.8 mm to (251.8, 77.4), turned to -90 degrees
- moved SW2 104.6 mm to (249.1, 77.3), turned to 90 degrees
- moved D8 99.2 mm to (200.4, 82.5)
- moved D6 92.9 mm to (203.4, 72.6), turned to -90 degrees
- moved R8 83.5 mm to (198.4, 86.0)
- moved C9 82.7 mm to (200.4, 72.6), turned to -90 degrees
- moved R7 80.5 mm to (193.5, 87.0)
- moved D7 77.9 mm to (193.4, 83.9)
- moved R26 61.2 mm to (175.9, 90.0), turned to -90 degrees
- moved R24 58.6 mm to (175.1, 87.2), turned to 180 degrees
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Connections:
- net /NIVARA_BOARD/DRIVER_RS485/UART_IN renamed /NIVARA_BOARD/DRIVER_RS485/UART-
- net /NIVARA_BOARD/DRIVER_RS485/UART_OUT renamed /NIVARA_BOARD/DRIVER_RS485/UART+
- net /NIVARA_BOARD/RS485_A renamed /NIVARA_BOARD/RS485_A+
- net /NIVARA_BOARD/RS485_B renamed /NIVARA_BOARD/RS485_B-
- D8 pad 1: Net-(D7-A2) -> Net-(D7-A1)
- D8 pad 2: Net-(D7-A1) -> Net-(D7-A2)
- R1 pad 1: Net-(U3-GPIO48/SPICLK_N/SUBSPICLK_N_DIFF) -> Net-(U3-GPIO1/TOUCH1/ADC1_CH0)
- R2 pad 1: Net-(U3-GPIO45) -> Net-(U3-GPIO2/TOUCH2/ADC1_CH1)
- R7 pad 1: Net-(D7-A1) -> Net-(D7-A2)
- R8 pad 1: Net-(D7-A2) -> Net-(D7-A1)
- U10 pad 9: unconnected-(U10-EP-Pad9) -> GND
- U3 pad 12: unconnected-(U3-GPIO8/TOUCH8/ADC1_CH7/SUBSPICS1-Pad12) -> /NIVARA_BOARD/PNP_IN_2/PNP_OUT
- U3 pad 15: unconnected-(U3-GPIO3/TOUCH3/ADC1_CH2-Pad15) -> /NIVARA_BOARD/PNP_IN_1/PNP_OUT
- U3 pad 16: unconnected-(U3-GPIO46-Pad16) -> /NIVARA_BOARD/NPN_IN_2/NPN_OUT
- U3 pad 17: unconnected-(U3-GPIO9/TOUCH9/ADC1_CH8/FSPIHD/SUBSPIHD-Pad17) -> /NIVARA_BOARD/NPN_IN_1/NPN_OUT
- U3 pad 18: /NIVARA_BOARD/A_V_OUT/ESP_SEL_VOUT -> /NIVARA_BOARD/A_V_OUT/SDA_V
- U3 pad 20: /NIVARA_BOARD/A_V_OUT/SDA_V -> /NIVARA_BOARD/A_V_OUT/ESP_SEL_VOUT
- U3 pad 21: /NIVARA_BOARD/A_I_OUT/SCLK_C -> /NIVARA_BOARD/PNP_OUT_2/PNP_IN
- U3 pad 22: /NIVARA_BOARD/A_I_OUT/SDA_C -> /NIVARA_BOARD/PNP_OUT_1/PNP_IN
- U3 pad 23: /NIVARA_BOARD/PNP_OUT_1/PNP_IN -> /NIVARA_BOARD/NPN_OUT_2/NPN_IN
- U3 pad 24: /NIVARA_BOARD/PNP_OUT_2/PNP_IN -> /NIVARA_BOARD/NPN_OUT_1/NPN_IN
- U3 pad 25: Net-(U3-GPIO48/SPICLK_N/SUBSPICLK_N_DIFF) -> /NIVARA_BOARD/A_I_OUT/SDA_C
- U3 pad 26: Net-(U3-GPIO45) -> /NIVARA_BOARD/A_I_OUT/SCLK_C
- U3 pad 28: /NIVARA_BOARD/D_IN_1/D_OUT -> /NIVARA_BOARD/RELAY1&2/ESP_RY1
- U3 pad 29: /NIVARA_BOARD/D_IN_2/D_OUT -> /NIVARA_BOARD/RELAY1&2/ESP_RLY2
- U3 pad 30: /NIVARA_BOARD/RUN_STOP/D_OUT -> unconnected-(U3-SPIDQS/GPIO37/FSPIQ/SUBSPIQ-Pad30)
- U3 pad 32: /NIVARA_BOARD/NPN_IN_1/NPN_OUT -> unconnected-(U3-MTCK/GPIO39/CLK_OUT3/SUBSPICS1-Pad32)
- U3 pad 33: /NIVARA_BOARD/NPN_IN_2/NPN_OUT -> unconnected-(U3-MTDO/GPIO40/CLK_OUT2-Pad33)
- U3 pad 34: /NIVARA_BOARD/NPN_OUT_1/NPN_IN -> unconnected-(U3-MTDI/GPIO41/CLK_OUT1-Pad34)
- U3 pad 35: /NIVARA_BOARD/NPN_OUT_2/NPN_IN -> unconnected-(U3-MTMS/GPIO42-Pad35)
- U3 pad 38: /NIVARA_BOARD/RELAY1&2/ESP_RY1 -> Net-(U3-GPIO2/TOUCH2/ADC1_CH1)
- U3 pad 39: /NIVARA_BOARD/RELAY1&2/ESP_RLY2 -> Net-(U3-GPIO1/TOUCH1/ADC1_CH0)
- U3 pad 4: /NIVARA_BOARD/4-20mA_IN/ESP_4-20_IN -> /NIVARA_BOARD/A_0-32_IN/A_V_OUT
- U3 pad 5: /NIVARA_BOARD/A_0-32_IN/A_V_OUT -> /NIVARA_BOARD/A_0-10_IN/A_V_OUT
- U3 pad 6: /NIVARA_BOARD/A_0-10_IN/A_V_OUT -> /NIVARA_BOARD/4-20mA_IN/ESP_4-20_IN
- U3 pad 7: unconnected-(U3-GPIO7/TOUCH7/ADC1_CH6-Pad7) -> /NIVARA_BOARD/RUN_STOP/D_OUT
- U3 pad 8: /NIVARA_BOARD/PNP_IN_1/PNP_OUT -> /NIVARA_BOARD/D_IN_2/D_OUT
- U3 pad 9: /NIVARA_BOARD/PNP_IN_2/PNP_OUT -> /NIVARA_BOARD/D_IN_1/D_OUT
- U5 pad 8: Net-(D7-A2) -> Net-(D7-A1)
- U5 pad 9: Net-(D7-A1) -> Net-(D7-A2)
Routing:
- net +3.3V: track 8.40 -> 212.7 mm, vias 112 -> 149
- net /NIVARA_BOARD/A_V_OUT/ESP_SEL_VOUT: track 0.00 -> 96.6 mm, vias 0 -> 1
- net /NIVARA_BOARD/A_V_OUT/SDA_V: track 0.00 -> 91.3 mm
- net /NIVARA_BOARD/A_V_OUT/SCLK_V: track 0.00 -> 88.8 mm
- net /NIVARA_BOARD/NPN_IN_1/NPN_OUT: track 5.30 -> 81.7 mm
- net /NIVARA_BOARD/A_I_OUT/SDA_C: track 4.68 -> 81.0 mm, vias 0 -> 2
- net /NIVARA_BOARD/A_I_OUT/SCLK_C: track 2.55 -> 76.1 mm, vias 0 -> 2
- net /NIVARA_BOARD/NPN_IN_2/NPN_OUT: track 5.30 -> 77.1 mm
- net /NIVARA_BOARD/RS485_A+: track 0.00 -> 70.9 mm, vias 0 -> 1
- net /NIVARA_BOARD/RS485_B-: track 0.00 -> 69.0 mm, vias 0 -> 1
- net Earth: track 34.5 -> 99.9 mm, vias 131 -> 120
- net /NIVARA_BOARD/PNP_IN_1/PNP_OUT: track 2.93 -> 63.4 mm
- net VCC: track 119.0 -> 179.4 mm, vias 23 -> 49
- net /NIVARA_BOARD/PNP_IN_2/PNP_OUT: track 3.00 -> 59.2 mm, vias 0 -> 2
- net /NIVARA_BOARD/RELAY1&2/ESP_RY1: track 0.00 -> 54.6 mm, vias 0 -> 2
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Other:
- board text added: "D2"
- board text added: "D7"
- board text added: "R51"
- board text added: "R52"
