File: Nivara_PCB/Nivara_PCB/Nivara_PCB.kicad_sch (KiCad schematic)
At the start: 23 parts, among them CN1 ANALOG_IN, CN2 RELAY, J1 AUXILIAR, P1 NPN_IN, P2 PNP_IN, P3 D_IN, P4 RUN/STOP, P5 NPN_OUT, P6 PNP_OUT, P7 RS485, P8 ANALOG_OUT., U1 2.54-2*2, U2 FUENTE IN

Commit message: Saved changes to Nivara PCB files
Parts:
- added D33: SMAJ33A, PCM_Diode_SMD_AKL:D_SMA, symbol EasyEDA:SMAJ33A
- added F2: BSMD1812-150-33V, EasyEDA:F1812, symbol EasyEDA:BSMD1812-150-33V
- added U20: FUENTE EX, EasyEDA:CONN-TH_XY126V-5.0-2P, symbol EasyEDA:XY126V-5.0-2P
Connections:
- net GND: no longer P4.2
- new net: F2.1, U20.1
- new net Earth: D33.2 (A), P4.2, U20.2
- new net VDD: D33.1 (K), F2.2

Commit message: PCB casi terminado.
Connections:
- net NIVARA_BOARD/RS485_A renamed NIVARA_BOARD/RS485_A+
- net NIVARA_BOARD/RS485_B renamed NIVARA_BOARD/RS485_B-
Other:
- sheet NIVARA_BOARD ports: added RS485_A+, RS485_B-; removed RS485_A, RS485_B
Changed lines of the file:
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@@
-			)
-		)
-		(pin "RS485_A" bidirectional
-			(at 116.84 81.28 0)
-			(effects
-				(font
-					(size 1.27 1.27)
-				)
-				(justify right)
-			)
-		)
-		(pin "RS485_B" bidirectional
-			(at 116.84 83.82 0)
-			(effects
-				(font
-					(size 1.27 1.27)
-				)
-				(justify right)
 			)
 		)
@@
 			)
 		)
+		(pin "RS485_A+" bidirectional
+			(at 116.84 81.28 0)
+			(effects
+				(font
+					(size 1.27 1.27)
+				)
+				(justify right)
+			)
+		)
+		(pin "RS485_B-" bidirectional
+			(at 116.84 83.82 0)
+			(effects
+				(font
+					(size 1.27 1.27)
+				)
+				(justify right)
+			)
+		)
