File: Nivara_PCB/Nivara_PCB/D_IN.kicad_sch (KiCad schematic)
At the start: 4 parts, among them U12 LTV-357T

Commit message: TERMINACIONES Y AJUSTES FINALES
Parts:
- removed D20: IR26-21C_L110_TR8, LED_SMD:LED_1206_3216Metric, symbol LED:IR26-21C_L110_TR8
- added D22: LED, LED_SMD:LED_0603_1608Metric, symbol EasyEDA:LED
- R33: renamed from R27; LCSC Part (none) -> C21190; Part # (none) -> 0603WAF1001T5E
- R34: renamed from R28; LCSC Part (none) -> C245910; Part # (none) -> RC0603FR-07140RL
- U14: renamed from U12; LCSC Part (none) -> C119091; Part # (none) -> LTV-357T-C
Connections:
- net D_OUT: now also D22.1 (K)
- net at R34.2: now also D22.2 (A)
