File: Nivara_PCB/Nivara_PCB/PNP_OUT.kicad_sch (KiCad schematic)
At the start: 8 parts, among them Q2 AO3407A, U9 LTV-357T

Commit message: TERMINACIONES Y AJUSTES FINALES
Parts:
- removed D16: IR26-21C_L110_TR8, LED_SMD:LED_1206_3216Metric, symbol LED:IR26-21C_L110_TR8
- added D16: LED, LED_SMD:LED_0603_1608Metric, symbol EasyEDA:LED
- D15: LCSC Part (none) -> C193342; Part # (none) -> PMEG4010CEH,115
- Q2: LCSC Part (none) -> C15155; Part # (none) -> AO3407A
- R21: renamed from R17; LCSC Part (none) -> C22775; Part # (none) -> 0603WAF1000T5E
- R22: renamed from R18; LCSC Part (none) -> C22775; Part # (none) -> 0603WAF1000T5E
- R23: renamed from R19; LCSC Part (none) -> C25803; Part # (none) -> 0603WAF1003T5E
- R24: renamed from R20; LCSC Part (none) -> C22843; Part # (none) -> 0603WAF1501T5E
- U11: renamed from U9; LCSC Part (none) -> C119091; Part # (none) -> LTV-357T-C
Connections:
- net Earth: now also R24.2
- net PNP_OUT: now also D16.2 (A); no longer R24.1
- new net: D16.1 (K), R24.1
Other:
- moved on the sheet: R24
