File: Nivara_PCB/Nivara_PCB/RELAY1&2.kicad_sch (KiCad schematic)
At the start: 3 parts, among them K1 SRA-24VDC-CL, K2 SRA-24VDC-CL, U11 LK1802

Commit message: TERMINACIONES Y AJUSTES FINALES
Parts:
- added D20, D21: LED, LED_SMD:LED_0603_1608Metric, symbol EasyEDA:LED
- added R31, R32: 1.5k, PCM_Resistor_SMD_AKL:R_0603_1608Metric, symbol EasyEDA:R_0603
- K1: renamed from K2; Part # (none) -> SRA-24VDC-CL
- K2: renamed from K1; Part # (none) -> SRA-24VDC-CL
- U13: renamed from U11; Part # (none) -> LK1802
Connections:
- net VCC: now also D20.2 (A), D21.2 (A)
- net at K1.4, U13.1 (1C): now also R31.2
- net at K2.3, U13.6 (2C): now also R32.2
- new net: D20.1 (K), R31.1
- new net: D21.1 (K), R32.1
Other:
- moved on the sheet: K1
