File: Nivara_PCB/PCB_USB/PCB_USB.kicad_pcb (KiCad board)
At the start: 2 copper layers, 47 x 13 mm, 6 parts, among them J1 PINHD_2x2_Male, U1 GT-USB-7010ASV

Commit message: Cambios en el PCB del USB.
Parts:
- moved J1 7.74 mm to (98.7, 93.8)
Routing:
- net /D-: track 38.4 -> 30.6 mm
- net /D+: track 38.9 -> 31.3 mm
Other:
- board size 47 x 13 mm -> 39.8 x 13 mm
Changed lines of the file:
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@@
 	(footprint "Connector_PinHeader_2.54mm:PinHeader_2x02_P2.54mm_Vertical"
 		(layer "F.Cu")
-		(at 90.96 93.96)
+		(at 98.7 93.76)
 		(descr "Through hole straight pin header, 2x02, 2.54mm pitch, double rows")
 		(tags "Through hole pin header THT 2x02 2.54mm double row")
@@
 		)
 		(embedded_fonts no)
-		(model "${KICAD9_3DMODEL_DIR}/Connector_PinHeader_2.54mm.3dshapes/PinHeader_2x02_P2.54mm_Vertical.step"
+		(model "${KICAD9_3DMODEL_DIR}/Connector_PinHeader_2.54mm.3dshapes/PinHeader_2x02_P2.54mm_Horizontal.wrl"
 			(offset
 				(xyz 0 0 0)
@@
 		)
 		(embedded_fonts no)
-		(model "${KICAD_3RD_PARTY}/EasyEDA.3dshapes/USB-C-SMD_G-SWITCH_GT-USB-7010ASV.wrl"
+		(model "${EASY_EDA}/USB-C-SMD_G-SWITCH_GT-USB-7010ASV.wrl"
 			(offset
-				(xyz 0 -1.05 1.5)
+				(xyz 0 -1.05 0)
 			)
 			(scale
@@
 			)
 			(rotate
-				(xyz 0 0 0)
+				(xyz -0 -0 -0)
 			)
 		)
@@
 	)
 	(gr_rect
-		(start 88 89)
+		(start 95.2 89)
 		(end 135 102)
 		(stroke
@@
 		(fill no)
 		(layer "Edge.Cuts")
-	)
-	(dimension
-		(type orthogonal)
-		(layer "F.Cu")
-		(pts
-			(xy 135 102) (xy 88 102)
-		)
-		(height 4.29)
-		(orientation 0)
-		(format
-			(prefix "")
-			(suffix "")
-			(units 3)
-			(units_format 0)
-			(precision 4)
-			(suppress_zeroes yes)
-		)
-		(style
-			(thickness 0.2)
-			(arrow_length 1.27)
-			(text_position_mode 0)
-			(arrow_direction outward)
-			(extension_height 0.58642)
-			(extension_offset 0.5)
-			(keep_text_aligned yes)
-		)
-		(gr_text "47"
-			(at 111.5 104.49 0)
-			(layer "F.Cu")
-			(effects
-				(font
-					(size 1.5 1.5)
-					(thickness 0.3)
-				)
-			)
-		)
 	)
 	(segment
@@
 	)
 	(segment
-		(start 94.775 95.225)
-		(end 93.5 96.5)
+		(start 102.315 95.225)
+		(end 101.24 96.3)
 		(width 0.2)
 		(layer "F.Cu")
@@
 	)
 	(segment
-		(start 129.0075 95.225)
-		(end 94.775 95.225)
+		(start 129.0325 95.25)
+		(end 129.0075 95.225)
 		(width 0.2)
 		(layer "F.Cu")
@@
 	)
 	(segment
-		(start 129.0325 95.25)
-		(end 129.0075 95.225)
+		(start 129.0075 95.225)
+		(end 102.315 95.225)
 		(width 0.2)
 		(layer "F.Cu")
@@
 	)
 	(segment
-		(start 94.29 94.75)
-		(end 93.5 93.96)
+		(start 129.0325 94.75)
+		(end 102.23 94.75)
 		(width 0.2)
 		(layer "F.Cu")
@@
 	)
 	(segment
-		(start 129.0325 94.75)
-		(end 94.29 94.75)
+		(start 102.23 94.75)
+		(end 101.24 93.76)
 		(width 0.2)
 		(layer "F.Cu")
@@
 		(polygon
 			(pts
-				(xy 88 89) (xy 135 89) (xy 135 102) (xy 88 102)
+				(xy 95.2 89) (xy 135 89) (xy 135 102) (xy 95.2 102)
 			)
 		)
@@
 		(polygon
 			(pts
-				(xy 135 89) (xy 135 102) (xy 88 102) (xy 88 89)
-			)
-		)
+				(xy 135 89) (xy 135 102) (xy 95.2 102) (xy 95.2 89)
+			)
+		)

Commit message: Change.
Parts:
- moved J1 3.82 mm to (101.2, 96.7), turned to 180 degrees
- moved R5 0.27 mm to (125.4, 96.7)
Connections:
- J1 pad 1: +5V -> /D+
- J1 pad 2: /D+ -> +5V
- J1 pad 3: GND -> /D-
- J1 pad 4: /D- -> GND
Routing:
- net /D-: track 30.6 -> 31.0 mm, vias 0 -> 2
- net GND: vias 0 -> 401

Commit message: Dimensiones.
Parts:
- moved J1 6.20 mm to (107.4, 96.5)
Routing:
- net /D-: track 31.0 -> 24.8 mm
- net /D+: track 30.9 -> 24.7 mm
- net GND: vias 401 -> 311
Other:
- board size 39.8 x 13 mm -> 33.4 x 13 mm

Commit message: Terminaciones de las dimensiones.
Other:
- board size 33.4 x 13 mm -> 33.4 x 18 mm
Changed lines of the file:
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@@
 	)
 	(gr_rect
-		(start 101.6 89)
-		(end 135 102)
+		(start 101.6 86.5)
+		(end 135 104.5)
 		(stroke
 			(width 0.05)
@@
 		(fill no)
 		(layer "Edge.Cuts")
-	)
-	(dimension
-		(type orthogonal)
-		(layer "F.Cu")
-		(pts
-			(xy 135 102) (xy 101.6 102)
-		)
-		(height 4.3)
-		(orientation 0)
-		(format
-			(prefix "")
-			(suffix "")
-			(units 3)
-			(units_format 0)
-			(precision 4)
-			(suppress_zeroes yes)
-		)
-		(style
-			(thickness 0.2)
-			(arrow_length 1.27)
-			(text_position_mode 0)
-			(arrow_direction outward)
-			(extension_height 0.58642)
-			(extension_offset 0.5)
-			(keep_text_aligned yes)
-		)
-		(gr_text "33.4"
-			(at 118.3 104.5 0)
-			(layer "F.Cu")
-			(effects
-				(font
-					(size 1.5 1.5)
-					(thickness 0.3)
-				)
-			)
-		)
 	)
 	(segment
@@
 		(polygon
 			(pts
-				(xy 101.6 89) (xy 135 89) (xy 135 102) (xy 101.6 102)
+				(xy 101.6 86.5) (xy 135 86.5) (xy 135 104.5) (xy 101.6 104.5)
 			)
 		)
@@
 		(polygon
 			(pts
-				(xy 135 89) (xy 135 102) (xy 101.6 102) (xy 101.6 89)
+				(xy 135 86.5) (xy 135 104.5) (xy 101.6 104.5) (xy 101.6 86.5)
 			)
 		)

Commit message: S.
Parts:
- moved J1 0.36 mm to (107.4, 96.9)
Changed lines of the file:
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@@
 	(footprint "Connector_PinHeader_2.54mm:PinHeader_2x02_P2.54mm_Vertical"
 		(layer "F.Cu")
-		(at 107.375 96.54 180)
+		(at 107.375 96.9 180)
 		(descr "Through hole straight pin header, 2x02, 2.54mm pitch, double rows")
 		(tags "Through hole pin header THT 2x02 2.54mm double row")
@@
 	)
 	(segment
-		(start 107.835 94.135)
+		(start 129.0325 95.25)
+		(end 108.75 95.25)
+		(width 0.2)
+		(layer "F.Cu")
+		(net 7)
+	)
+	(segment
+		(start 108.75 95.25)
+		(end 107.86 94.36)
+		(width 0.2)
+		(layer "F.Cu")
+		(net 7)
+	)
+	(segment
+		(start 107.375 94.36)
 		(end 107.375 94.135)
 		(width 0.2)
@@
 	)
 	(segment
-		(start 108.95 95.25)
-		(end 107.835 94.135)
+		(start 107.86 94.36)
+		(end 107.375 94.36)
 		(width 0.2)
 		(layer "F.Cu")
@@
 		(net 7)
 	)
-	(segment
-		(start 129.0325 95.25)
-		(end 108.95 95.25)
-		(width 0.2)
-		(layer "F.Cu")
-		(net 7)
-	)
 	(via
 		(at 127.6 96.325)
@@
 	)
 	(segment
-		(start 129.0325 95.75)
-		(end 128.102499 95.75)
+		(start 128.102499 95.75)
+		(end 128.077499 95.725)
 		(width 0.2)
 		(layer "F.Cu")
@@
 	)
 	(segment
-		(start 128.102499 95.75)
-		(end 128.077499 95.725)
+		(start 107.825 96.675)
+		(end 107.775 96.675)
 		(width 0.2)
 		(layer "F.Cu")
@@
 	)
 	(segment
-		(start 107.970698 96.675)
-		(end 107.775 96.675)
+		(start 128.077499 95.725)
+		(end 108.775 95.725)
 		(width 0.2)
 		(layer "F.Cu")
@@
 	)
 	(segment
-		(start 108.920698 95.725)
-		(end 107.970698 96.675)
+		(start 129.0325 95.75)
+		(end 128.102499 95.75)
 		(width 0.2)
 		(layer "F.Cu")
@@
 	)
 	(segment
-		(start 130.01 95.75)
-		(end 129.0325 95.75)
+		(start 108.775 95.725)
+		(end 107.825 96.675)
 		(width 0.2)
 		(layer "F.Cu")
@@
 	)
 	(segment
-		(start 128.077499 95.725)
-		(end 108.920698 95.725)
+		(start 130.01 95.75)
+		(end 129.0325 95.75)
 		(width 0.2)
 		(layer "F.Cu")

Commit message: PCB casi terminado.
Parts:
- moved J1 2.90 mm to (107.4, 94.0), turned to -90 degrees
Routing:
- net /D-: track 24.9 -> 30.2 mm
- net /D+: track 24.7 -> 25.5 mm
Changed lines of the file:
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@@
 	(footprint "Connector_PinHeader_2.54mm:PinHeader_2x02_P2.54mm_Vertical"
 		(layer "F.Cu")
-		(at 107.375 96.9 180)
+		(at 107.375 94 -90)
 		(descr "Through hole straight pin header, 2x02, 2.54mm pitch, double rows")
 		(tags "Through hole pin header THT 2x02 2.54mm double row")
 		(property "Reference" "J1"
-			(at 1.27 -2.380001 0)
+			(at 1.27 -2.380001 90)
 			(layer "F.SilkS")
 			(hide yes)
@@
 		)
 		(property "Value" "PINHD_2x2_Male"
-			(at 1.27 4.92 0)
+			(at 1.27 4.92 90)
 			(layer "F.Fab")
 			(effects
@@
 		)
 		(property "Datasheet" ""
-			(at 0 0 0)
+			(at 0 0 90)
 			(layer "F.Fab")
 			(hide yes)
@@
 		)
 		(property "Description" "Pin Header male with pin space 2.54mm. Pin Count -4"
-			(at 0 0 0)
+			(at 0 0 90)
 			(layer "F.Fab")
 			(hide yes)
@@
 		(attr through_hole)
 		(fp_line
-			(start 3.92 -1.38)
+			(start -1.38 3.92)
 			(end 3.92 3.92)
 			(stroke
@@
 		)
 		(fp_line
-			(start 1.27 1.27)
-			(end 1.27 -1.38)
+			(start -1.38 1.27)
+			(end -1.38 3.92)
 			(stroke
 				(width 0.12)
@@
 		)
 		(fp_line
-			(start 1.27 -1.38)
-			(end 3.92 -1.38)
+			(start -1.38 1.27)
+			(end 1.27 1.27)
 			(stroke
 				(width 0.12)
@@
 		)
 		(fp_line
-			(start -1.379999 0)
-			(end -1.38 -1.38)
+			(start 1.27 1.27)
+			(end 1.27 -1.38)
 			(stroke
 				(width 0.12)
@@
 		)
 		(fp_line
-			(start -1.38 3.92)
-			(end 3.92 3.92)
+			(start -1.379999 0)
+			(end -1.38 -1.38)
 			(stroke
 				(width 0.12)
@@
 		)
 		(fp_line
-			(start -1.38 1.27)
-			(end 1.27 1.27)
+			(start -1.38 -1.38)
+			(end 0 -1.379999)
 			(stroke
 				(width 0.12)
@@
 		)
 		(fp_line
-			(start -1.38 1.27)
-			(end -1.38 3.92)
+			(start 1.27 -1.38)
+			(end 3.92 -1.38)
 			(stroke
 				(width 0.12)
@@
 		)
 		(fp_line
-			(start -1.38 -1.38)
-			(end 0 -1.379999)
+			(start 3.92 -1.38)
+			(end 3.92 3.92)
 			(stroke
 				(width 0.12)
@@
 		)
 		(fp_line
-			(start 4.32 4.32)
-			(end 4.32 -1.77)
+			(start -1.77 4.32)
+			(end 4.32 4.32)
 			(stroke
 				(width 0.05)
@@
 		)
 		(fp_line
-			(start 4.32 -1.77)
-			(end -1.77 -1.77)
+			(start 4.32 4.32)
+			(end 4.32 -1.77)
 			(stroke
 				(width 0.05)
@@
 		)
 		(fp_line
-			(start -1.77 4.32)
-			(end 4.32 4.32)
+			(start -1.77 -1.77)
+			(end -1.77 4.32)
 			(stroke
 				(width 0.05)
@@
 		)
 		(fp_line
-			(start -1.77 -1.77)
-			(end -1.77 4.32)
+			(start 4.32 -1.77)
+			(end -1.77 -1.77)
 			(stroke
 				(width 0.05)
@@
 		)
 		(fp_line
-			(start 3.81 3.81)
-			(end -1.27 3.81)
+			(start -1.27 3.81)
+			(end -1.270001 0)
 			(stroke
 				(width 0.1)
@@
 		)
 		(fp_line
-			(start 3.81 -1.27)
-			(end 3.81 3.81)
+			(start 3.81 3.81)
+			(end -1.27 3.81)
 			(stroke
 				(width 0.1)
@@
 		)
 		(fp_line
-			(start 0 -1.270001)
-			(end 3.81 -1.27)
+			(start -1.270001 0)
+			(end 0 -1.270001)
 			(stroke
 				(width 0.1)
@@
 		)
 		(fp_line
-			(start -1.27 3.81)
-			(end -1.270001 0)
+			(start 3.81 -1.27)
+			(end 3.81 3.81)
 			(stroke
 				(width 0.1)
@@
 		)
 		(fp_line
-			(start -1.270001 0)
-			(end 0 -1.270001)
+			(start 0 -1.270001)
+			(end 3.81 -1.27)
 			(stroke
 				(width 0.1)
@@
 		)
 		(fp_text user "${REFERENCE}"
-			(at 1.27 1.27 90)
+			(at 1.27 1.27 0)
 			(layer "F.Fab")
 			(effects
@@
 		)
 		(pad "1" thru_hole rect
-			(at 0 0 180)
+			(at 0 0 270)
 			(size 1.7 1.7)
 			(drill 1)
@@
 		)
 		(pad "2" thru_hole circle
-			(at 2.54 0 180)
+			(at 2.54 0 270)
 			(size 1.7 1.7)
 			(drill 1)
@@
 		)
 		(pad "3" thru_hole circle
-			(at 0 2.54 180)
+			(at 0 2.54 270)
 			(size 1.7 1.7)
 			(drill 1)
@@
 		)
 		(pad "4" thru_hole circle
-			(at 2.54 2.54 180)
+			(at 2.54 2.54 270)
 			(size 1.7 1.7)
 			(drill 1)
@@
 	)
 	(segment
+		(start 129.0325 95.25)
+		(end 109.45 95.25)
+		(width 0.2)
+		(layer "F.Cu")
+		(net 7)
+	)
+	(segment
 		(start 128.1115 96.325)
 		(end 128.1115 96.299)
@@
 	)
 	(segment
-		(start 129.0325 95.25)
-		(end 108.75 95.25)
+		(start 105.5 92.5)
+		(end 104.835 93.165)
+		(width 0.2)
+		(layer "F.Cu")
+		(net 7)
+	)
+	(segment
+		(start 104.835 93.165)
+		(end 104.835 94)
 		(width 0.2)
 		(layer "F.Cu")
@@
 	)
 	(segment
-		(start 108.75 95.25)
-		(end 107.86 94.36)
+		(start 108.8 92.8)
+		(end 108.5 92.5)
 		(width 0.2)
 		(layer "F.Cu")
@@
 	)
 	(segment
-		(start 107.375 94.36)
-		(end 107.375 94.135)
+		(start 109.45 95.25)
+		(end 108.8 94.6)
 		(width 0.2)
 		(layer "F.Cu")
@@
 	)
 	(segment
-		(start 128.9835 96.299)
-		(end 129.0325 96.25)
+		(start 108.5 92.5)
+		(end 105.5 92.5)
 		(width 0.2)
 		(layer "F.Cu")
@@
 	)
 	(segment
-		(start 107.86 94.36)
-		(end 107.375 94.36)
+		(start 128.9835 96.299)
+		(end 129.0325 96.25)
 		(width 0.2)
 		(layer "F.Cu")
@@
 		(net 7)
 	)
+	(segment
+		(start 108.8 94.6)
+		(end 108.8 92.8)
+		(width 0.2)
+		(layer "F.Cu")
+		(net 7)
+	)
 	(via
 		(at 127.6 96.325)
@@
 	)
 	(segment
-		(start 129.0325 94.75)
-		(end 129.9045 94.75)
+		(start 128.077499 95.725)
+		(end 109.225 95.725)
 		(width 0.2)
 		(layer "F.Cu")
@@
 	)
 	(segment
-		(start 129.9045 94.75)
-		(end 130.24 95.0855)
+		(start 129.0325 94.75)
+		(end 129.9045 94.75)
 		(width 0.2)
 		(layer "F.Cu")
@@
 	)
 	(segment
-		(start 128.102499 95.75)
-		(end 128.077499 95.725)
+		(start 129.9045 94.75)
+		(end 130.24 95.0855)
 		(width 0.2)
 		(layer "F.Cu")
@@
 	)
 	(segment
-		(start 130.24 95.52)
-		(end 130.01 95.75)
+		(start 129.0325 95.75)
+		(end 128.102499 95.75)
 		(width 0.2)
 		(layer "F.Cu")
@@
 	)
 	(segment
-		(start 107.825 96.675)
-		(end 107.775 96.675)
+		(start 130.24 95.52)
+		(end 130.01 95.75)
 		(width 0.2)
 		(layer "F.Cu")
@@
 	)
 	(segment
-		(start 128.077499 95.725)
-		(end 108.775 95.725)
+		(start 128.102499 95.75)
+		(end 128.077499 95.725)
 		(width 0.2)
 		(layer "F.Cu")
@@
 	)
 	(segment
-		(start 129.0325 95.75)
-		(end 128.102499 95.75)
+		(start 109.225 95.725)
+		(end 107.5 94)
 		(width 0.2)
 		(layer "F.Cu")
@@
 	)
 	(segment
-		(start 108.775 95.725)
-		(end 107.825 96.675)
+		(start 107.5 94)
+		(end 107.375 94)
 		(width 0.2)
 		(layer "F.Cu")

Commit message: TERMINACIONES Y AJUSTES FINALES
Parts:
- removed D2: IR26-21C_L110_TR8, LED_SMD:LED_1206_3216Metric
- added D5: LED, LED_SMD:LED_0603_1608Metric, F.Cu at (124.8, 99.7)
- moved R6 5.68 mm to (124.8, 97.5)
- moved R5 1.02 mm to (124.9, 95.8)
- moved R7 0.79 mm to (124.9, 93.2)
- moved J1 0.15 mm to (107.3, 94.2)
Connections:
- J1 pad 1: /D+ -> /D-
- J1 pad 3: /D- -> /D+
Routing:
- net /D-: track 30.2 -> 24.6 mm, vias 2 -> 0
- net /D+: track 25.5 -> 28.7 mm
- net +5V: track 11.1 -> 9.34 mm
- net Net-(U1-CC2): track 2.80 -> 3.59 mm
- net Net-(U1-CC1): track 3.11 -> 3.73 mm
- net GND: vias 311 -> 333
